File: kicad/nahs-Bricks-Interface_v4.0_r1/nahs-Bricks-Interface_v4.0_r1.kicad_pcb (KiCad board)
At the start: 2 copper layers, 63.6 x 105.4 mm, 37 parts, among them J1 Brick-Interface-V4, J2 Brick-Interface-V4, J3 TE_292304-1, J4 TE_292303-1, SW1 K3-2336S-F1, SW2 K3-2336S-F1, SW3 K3-2336S-F1, SW4 Taster_3301, U1 SL2.1A, U2 CP2102N-A02-GQFN20R, U3 FT232RL, Y1 12MHz

Commit message: v4.0 r1 Board done
Parts:
- removed FID1, FID2, FID3: Fiducial_1mm_Mask2mm, Fiducial:Fiducial_1mm_Mask2mm
- removed LOGOB, LOGOF: x17mm, no_brick_logo:x17mm
Connections:
- J3 pad 5: unconnected-(J3-Pad5) -> Net-(J3-Pad5)
- J4 pad 5: unconnected-(J4-Pad5) -> Net-(J3-Pad5)
Routing:
- net Net-(J3-Pad5): track 0.00 -> 41.4 mm
- net unconnected-(J4-Pad5): track 13.1 -> 0.00 mm
- net unconnected-(J3-Pad5): track 12.0 -> 0.00 mm
