File: kicad/nahs-Bricks-Interface_v4.0_r1/nahs-Bricks-Interface_v4.0_r1.kicad_sch (KiCad schematic)
At the start: 32 parts, among them J1 Brick-Interface-V4, J2 Brick-Interface-V4, J3 TE_292304-1, J4 TE_292303-1, SW1 K3-2336S-F1, SW2 K3-2336S-F1, SW3 K3-2336S-F1, SW4 Taster_3301, U1 SL2.1A, U2 CP2102N-A02-GQFN20R, U3 FT232RL, Y1 12MHz

Commit message: v4.0 r1 Board done
Connections:
- net at J4.5 (Shield): now also J3.5 (Shield)
Changed lines of the file:
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@@
+    (stroke (width 0) (type default) (color 0 0 0 0))
+  )
+  (wire (pts (xy 134.62 44.45) (xy 134.62 76.2))
     (stroke (width 0) (type default) (color 0 0 0 0))
   )
@@
   )
   (wire (pts (xy 207.01 88.9) (xy 205.74 88.9))
+    (stroke (width 0) (type default) (color 0 0 0 0))
+  )
+  (wire (pts (xy 143.51 43.18) (xy 143.51 44.45))
     (stroke (width 0) (type default) (color 0 0 0 0))
   )
@@
     (stroke (width 0) (type default) (color 0 0 0 0))
   )
+  (wire (pts (xy 143.51 44.45) (xy 134.62 44.45))
+    (stroke (width 0) (type default) (color 0 0 0 0))
+  )
   (wire (pts (xy 101.6 24.13) (xy 105.41 24.13))
     (stroke (width 0) (type default) (color 0 0 0 0))
@@
     (stroke (width 0) (type default) (color 0 0 0 0))
   )
+  (wire (pts (xy 134.62 76.2) (xy 143.51 76.2))
+    (stroke (width 0) (type default) (color 0 0 0 0))
+  )
