File: kicad/nahs-Bricks-Interface_v4.0_r2/nahs-Bricks-Interface_v4.0_r2.kicad_pcb (KiCad board)
At the start: 2 copper layers, 63.6 x 105.4 mm, 43 parts, among them J1 Brick-Interface-V4, J2 Brick-Interface-V4, J3 TE_292304-1, J4 TE_292303-1, SW1 K3-2336S-F1, SW2 K3-2336S-F1, SW3 K3-2336S-F1, SW4 Taster_4545, U1 SL2.1A, U2 CP2102N-A02-GQFN20R, Y1 12MHz

Commit message: changed colors of LEDs
Parts:
- D2: value RED -> BLUE
- D3: value GREEN -> YELLOW
Changed lines of the file:
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@@
     (property "Sheetname" "")
     (property "Storage" "MAG4")
-    (property "StorageDesc" "LED Green")
+    (property "StorageDesc" "LED Yellow")
     (attr smd)
     (fp_text reference "D3" (at 2.4 0 180) (layer "F.SilkS")
       (effects (font (size 1 1) (thickness 0.15)))
     )
-    (fp_text value "GREEN" (at 0 1.65 90) (layer "F.Fab") hide
+    (fp_text value "YELLOW" (at 0 1.65 90) (layer "F.Fab") hide
       (effects (font (size 1 1) (thickness 0.15)))
     )
@@
     (property "Sheetname" "")
     (property "Storage" "MAG4")
-    (property "StorageDesc" "LED OrangeRed")
+    (property "StorageDesc" "LED Blue")
     (attr smd)
     (fp_text reference "D2" (at 2.4 0 180) (layer "F.SilkS")
       (effects (font (size 1 1) (thickness 0.15)))
     )
-    (fp_text value "RED" (at 0 1.65 90) (layer "F.Fab") hide
-      (effects (font (size 1 1) (thickness 0.15)))
-    )
+    (fp_text value "BLUE" (at 0 1.65 90) (layer "F.Fab") hide
+      (effects (font (size 1 1) (thickness 0.15)))
+    )
